File: brine_electronics/Brine Mainboard/_autosave-Brine.kicad_pcb (KiCad board)
At the start: 2 copper layers, 30.5 x 42.7 mm, 17 parts, among them J1 Conn_01x02_Socket, U1 XIAO-ESP32-S3-SMD, U2 VL53L1CXV0FY1

Commit message: Updated electronics/enclosure designs
Parts:
- J1: moved to B.Cu
- moved J1 2.00 mm to (141.4, 105.8), turned to 0 degrees
Routing:
- net /Battery/BATT: track 26.1 -> 22.4 mm
