File: brine_electronics/Brine Mainboard/Brine.kicad_pcb (KiCad board)
At the start: 2 copper layers, 30.4 x 42.6 mm, 29 parts, among them J1 BATT, J2 BATT_CRG_GND, J3 BATT_CRG_BATT, J4 BATT_CRG_BATT, J5 BATT_CRG_GND, Q1 AO3407A, U1 XIAO-ESP32-S3-SMD, U2 VL53L1CXV0FY1, U3 LTC2954, U4 74AHCT1G125

Commit message: Updated production files 🏭
Routing:
- net GND: track 57.4 -> 53.5 mm, vias 12 -> 17
Other:
- board text added: "05/26/2026"
- board text added: "Version 07"
- board text removed: "04/18/26"
- board text removed: "Version 06"
Changed lines of the file:
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@@
 		)
 	)
-	(gr_text "Version 06"
+	(gr_text "Version 07"
 		(at 166.211572 109.500782 0)
 		(layer "B.SilkS")
@@
 		)
 	)
-	(gr_text "04/18/26"
+	(gr_text "05/26/2026"
 		(at 166.304688 111.009273 0)
 		(layer "B.SilkS")
@@
 			(font
 				(size 1 1)
-				(thickness 0.1)
+				(thickness 0.2)
+				(bold yes)
 			)
 			(justify left bottom mirror)
@@
 	)
 	(via
+		(at 144.981816 98.298005)
+		(size 0.6)
+		(drill 0.3)
+		(layers "F.Cu" "B.Cu")
+		(free yes)
+		(net "GND")
+	)
+	(via
+		(at 141.646821 91.207431)
+		(size 0.6)
+		(drill 0.3)
+		(layers "F.Cu" "B.Cu")
+		(free yes)
+		(net "GND")
+	)
+	(via
 		(at 141.967206 98.014829)
 		(size 0.6)
@@
 	)
 	(via
+		(at 141.821467 82.100911)
+		(size 0.6)
+		(drill 0.3)
+		(layers "F.Cu" "B.Cu")
+		(free yes)
+		(net "GND")
+	)
+	(via
 		(at 165.12302 92.518088)
 		(size 0.6)
@@
 		)
 		(filling no)
+		(net "GND")
+	)
+	(via
+		(at 154.426725 87.960785)
+		(size 0.6)
+		(drill 0.3)
+		(layers "F.Cu" "B.Cu")
+		(free yes)
+		(net "GND")
+	)
+	(via
+		(at 156.665911 95.463991)
+		(size 0.6)
+		(drill 0.3)
+		(layers "F.Cu" "B.Cu")
+		(free yes)
 		(net "GND")
 	)
@@
 	)
 	(segment
-		(start 149.86 74.93)
-		(end 148.322734 76.467266)
-		(width 0.2)
-		(layer "B.Cu")
-		(net "GND")
-	)
-	(segment
 		(start 138.43 83.82)
 		(end 138.43 83.07869)
@@
 		(start 157.48 100.33)
 		(end 153.947457 100.33)
-		(width 0.2)
-		(layer "B.Cu")
-		(net "GND")
-	)
-	(segment
-		(start 148.322734 76.467266)
-		(end 146.647404 76.467266)
 		(width 0.2)
 		(layer "B.Cu")
@@
 		(start 155.4 110.175)
 		(end 149.4 110.175)
-		(width 0.2)
+		(width 0.6)
 		(layer "F.Cu")
 		(net "/Button/BUTTON")
