File: brine_electronics/Brine Mainboard/brine_battery_monitor.kicad_sch (KiCad schematic)
At the start: 2 parts

Commit message: Implemented power latch circuit ⚡
Connections:
- net BATT renamed SYS_VBAT
Changed lines of the file:
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@@
 		)
 	)
-	(hierarchical_label "BATT"
+	(hierarchical_label "SYS_VBAT"
 		(shape output)
 		(at 100.33 101.6 180)

Commit message: Updated production files 🏭
Parts:
- R1: LCSC Part # (none) -> C17556
- R2: LCSC Part # (none) -> C25611
Changed lines of the file:
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@@
+			)
+		)
+		(property "Color" ""
+			(at 116.84 101.6 90)
+			(hide yes)
+			(show_name no)
+			(do_not_autoplace no)
+			(effects
+				(font
+					(size 1.27 1.27)
+				)
+			)
+		)
+		(property "LCSC Part #" "C17556"
+			(at 116.84 101.6 90)
+			(hide yes)
+			(show_name no)
+			(do_not_autoplace no)
+			(effects
+				(font
+					(size 1.27 1.27)
+				)
 			)
 		)
@@
 			(hide yes)
 			(show_name no)
+			(do_not_autoplace no)
+			(effects
+				(font
+					(size 1.27 1.27)
+				)
+			)
+		)
+		(property "Color" ""
+			(at 144.78 101.6 90)
+			(hide yes)
+			(show_name no)
+			(do_not_autoplace no)
+			(effects
+				(font
+					(size 1.27 1.27)
+				)
+			)
+		)
+		(property "LCSC Part #" "C25611"
+			(at 144.78 101.6 90)
+			(hide yes)
+			(show_name no)

Commit message: Updated electronics production files 🏭
Parts:
- R1: JLCPCB Part # (none) -> C17556; LCSC Part # C17556 -> (none)
- R2: JLCPCB Part # (none) -> C25611; LCSC Part # C25611 -> (none)
Changed lines of the file:
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@@
 			)
 		)
-		(property "LCSC Part #" "C17556"
+		(property "JLCPCB Part #" "C17556"
 			(at 116.84 101.6 90)
 			(hide yes)
@@
 			)
 		)
-		(property "LCSC Part #" "C25611"
+		(property "JLCPCB Part #" "C25611"
 			(at 144.78 101.6 90)
 			(hide yes)
